File: hardware/chaves.sch (EAGLE design)
At the start: 72 parts, among them IC1 40106N

Commit message: all done except ground plane
Parts:
- removed R1, R2, R3, R4, R5, R6: 10k, adafruit:R-US_0204/7
- added IN1, IN2: WQP-PJ301M-12_JACK, MusicThingModular:WQP-PJ301M-12_JACK
- added JP6, JP7: (no value), adafruit:PINHD-1X3CB
- added POT7, POT8: 10k, pot-alps:POT_USVERTICAL
Connections:
- removed net N$3 (its old number): C5.1, U$8.O
- removed net N$36: IC1F.I, LDR2.1, POT6.E, POT6.S, U$12.P
- removed net N$6 (its old number): C6.1, U$9.S
- new net N$23: IN1.2, POT7.A
- new net N$46: C10.2, U$11.O
- new net N$47: C10.1, C11.1, IC1E.I, POT5.E, POT5.S
- new net N$48: C11.2, U$11.S
- new net N$49: C13.2, U$12.S
- new net N$50: C12.2, U$12.O
- new net N$51: C12.1, C13.1, IC1F.I, POT6.E, POT6.S
- net GND: now also IN1.1, IN2.1, POT7.E, POT8.E; no longer R1.1, R2.1, R3.1, R4.1, R5.1, R6.1
- net N$1: now also C1.2; no longer C2.1
- net N$10: now also C6.2, U$9.O; no longer C10.1, U$11.S
- net N$11: now also C7.2, U$9.S; no longer C13.1, U$12.O
- net N$12: now also JP6.1, JP6.2, JP6.3, POT7.S; no longer C12.1, U$12.S
- net N$18: no longer R1.2
- net N$19: now also LDR1.1
- net N$2: now also C2.2; no longer C1.1
- net N$22: now also LDR2.1
- net N$27: no longer R2.2
- net N$30: no longer R3.2
- net N$31: now also C1.1, C2.1; no longer LDR1.1, U$7.P
- net N$32: now also C4.1, C5.1; no longer U$8.P
- net N$33: now also C6.1, C7.1; no longer U$9.P
- net N$34: now also C8.1, C9.1; no longer U$10.P
- net N$35: now also JP7.1, JP7.3, POT8.S; no longer IC1E.I, POT5.E, POT5.S, U$11.P
- net N$39: no longer R4.2
- net N$4: now also C5.2; no longer C4.1
- net N$42: no longer R5.2
- net N$45: no longer R6.2
- net N$5: now also C4.2, U$8.O; no longer C7.1, U$9.O
- net N$7: now also C8.2; no longer C9.1
- net N$8: now also C9.2; no longer C8.1
- net N$9: now also IN2.2, POT8.A; no longer C11.1, U$11.O
- net SS1: now also U$7.P; no longer C1.2, C2.2
- net SS2: now also U$8.P; no longer C4.2, C5.2
- net SS3: now also U$9.P; no longer C6.2, C7.2
- net SS4: now also U$10.P; no longer C8.2, C9.2
- net SS5: now also U$11.P; no longer C10.2, C11.2
- net SS6: now also U$12.P; no longer C12.2, C13.2
Other:
- moved on the sheet: C1, C10, C11, C12, C13, C2, C4, C5, C6, C7, C8, C9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

Commit message: Ground planed
Connections:
- removed net N$35: JP7.1, JP7.3, POT8.S
- new net N$25: JP7.1, JP7.2, JP7.3, POT8.S
Changed lines of the file:
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@@
 </segment>
 </net>
-<net name="N$35" class="0">
+<net name="N$25" class="0">
 <segment>
 <pinref part="JP7" gate="A" pin="3"/>
+<pinref part="JP7" gate="A" pin="2"/>
+<wire x1="193.04" y1="106.68" x2="195.58" y2="106.68" width="0.1524" layer="91"/>
+<pinref part="JP7" gate="A" pin="1"/>
+<wire x1="198.12" y1="106.68" x2="195.58" y2="106.68" width="0.1524" layer="91"/>
 <pinref part="POT8" gate="G$1" pin="S"/>
-<wire x1="193.04" y1="106.68" x2="195.58" y2="106.68" width="0.1524" layer="91"/>
 <wire x1="195.58" y1="106.68" x2="195.58" y2="114.3" width="0.1524" layer="91"/>
-<pinref part="JP7" gate="A" pin="1"/>
-<wire x1="195.58" y1="106.68" x2="198.12" y2="106.68" width="0.1524" layer="91"/>
 </segment>
 </net>
