File: v3/hardware/chaves.brd (EAGLE design)
At the start: 100 x 100 mm, 101 parts, among them IC1 40106N, J2 DCJ0202, T1 bc547, T2 bc547

Commit message: working on position board v3
Parts:
- moved D2 8.59 mm to (78.5, 91.5), turned to 90 degrees
- moved +5V 3.91 mm to (74.2, 69.2)
- moved JHSYNC 2.72 mm to (66.0, 80.5)
- moved JGND 2.61 mm to (66.5, 69.0)
- moved BJ 1.71 mm to (78.0, 75.0)
- moved JVCC1 1.56 mm to (86.0, 53.0)
- moved GJ 1.53 mm to (70.5, 75.0)
- moved JVSYNC 1.40 mm to (76.5, 80.5)
- moved IC1 1.12 mm to (70.5, 59.0)
- moved RJ 0.76 mm to (63.0, 75.0)
Other:
- board text added: "BLUE"
- board text added: "CHAV/ES - based on jonasbers.com/chav/"
- board text added: "G"
- board text added: "GREEN"
- board text added: "H"
- board text added: "IN1"
- board text added: "IN2"
- board text added: "IN3"
- board text added: "RED"
- board text added: "V"
- board text added: "VCO1"
- board text added: "VCO2"
- board text added: "VCO3"
- board text added: "VCO4"
- board text added: "VCO5"
- board text added: "VCO6"
- board text added: "pcb by luix github.com/Ttreintaysiete/chaves"
- board text added: "version 3"
- board text removed: "CHA/VES - based on jonasbers.com/chav/"
- board text removed: "ON"
